Commit message: add lidar sensor

File: origin_one_description/urdf/origin_one.urdf.xacro (robot description, xacro)
@@ -297,4 +297,54 @@
           <min>0.08</min>
           <max>100.0</max>
+          <resolution>0.01</resolution>
+        </range>
+        <noise type="gaussian">
+          <mean>0.0</mean>
+          <stddev>0.01</stddev>
+        </noise>
+      </lidar>
+      <alwaysOn>1</alwaysOn>
+      <visualize>true</visualize>
+    </sensor>
+  </gazebo>
+  <!-- 2D LiDAR for Nav2 (LaserScan) -->
+  <link name="scan_link">
+    <inertial>
+      <mass value="0.05"/>
+      <inertia ixx="0.0001" ixy="0.0" ixz="0.0" iyy="0.0001" iyz="0.0" izz="0.0001"/>
+    </inertial>
+    <visual name="visual">
+      <origin xyz="0 0 0" rpy="0 0 0"/>
+      <geometry>
+        <cylinder length="0.05" radius="0.05"/>
+      </geometry>
+      <material name="black">
+        <color rgba="1 1 1 1"/>
+      </material>
+    </visual>
+    <collision name="collision">
+      <origin xyz="0 0 0" rpy="0 0 0"/>
+      <geometry>
+        <cylinder length="0.05" radius="0.05"/>
+      </geometry>
+    </collision>
+  </link>
+  <gazebo reference="scan_link">
+    <sensor name="2d_lidar" type="gpu_lidar">
+      <topic>/scan</topic>
+      <gz_frame_id>scan_link</gz_frame_id>
+      <update_rate>10</update_rate>
+      <lidar>
+        <scan>
+          <horizontal>
+            <samples>360</samples>
+            <resolution>1.0</resolution>
+            <min_angle>-3.1415926</min_angle>
+            <max_angle>3.1415926</max_angle>
+          </horizontal>
+        </scan>
+        <range>
+          <min>0.12</min>
+          <max>30.0</max>
           <resolution>0.01</resolution>
         </range>
@@ -392,14 +442,16 @@
           <horizontal>
             <!-- Noise in degrees: https://github.com/gazebosim/gz-sensors/issues/325 -->
+            <!-- Reduced noise for more precise GPS -->
             <noise type="gaussian">
               <mean>0.0</mean>
-              <stddev>0.0001</stddev>
+              <stddev>0.00001</stddev>
             </noise>
           </horizontal>
           <vertical>
             <!-- Noise in degrees -->
+            <!-- Reduced noise for more precise GPS -->
             <noise type="gaussian">
               <mean>0.0</mean>
-              <stddev>0.0001</stddev>
+              <stddev>0.00001</stddev>
             </noise>
           </vertical>
@@ -421,5 +473,26 @@
   </link>
   <link name="imu_link">
-  </link>
+    <inertial>
+      <mass value="0.01"/>
+      <inertia ixx="0.0001" ixy="0.0" ixz="0.0" iyy="0.0001" iyz="0.0" izz="0.0001"/>
+    </inertial>
+  </link>
+  <gazebo reference="imu_link">
+    <sensor name="GazeboIMU" type="imu">
+      <always_on>1</always_on>
+      <update_rate>25.0</update_rate>
+      <visualize>true</visualize>
+      <topic>imu</topic>
+      <frame_id>imu_link</frame_id>
+      <ignition_frame_id>imu_link</ignition_frame_id>
+      <imu>
+        <orientation_reference_frame>
+          <localization>ENU</localization>
+        </orientation_reference_frame>
+      </imu>
+      <plugin filename="ignition-gazebo-imu-system" name="ignition::gazebo::systems::Imu">
+      </plugin>
+    </sensor>
+  </gazebo>
   <joint type="fixed" name="base_body">
     <origin xyz="0.0 0 ${groundClearance}" rpy="0 0 0"/>
@@ -478,4 +551,9 @@
     <origin xyz="-0.0505 0 0.212" rpy="0 0 0"/>
     <child link="gnss_link"/>
+    <parent link="main_body"/>
+  </joint>
+  <joint type="fixed" name="scan_joint">
+    <origin xyz="-0.05 0 0.3" rpy="0 0 0"/>
+    <child link="scan_link"/>
     <parent link="main_body"/>
   </joint>
